File: soic-16/soic-16.kicad_pcb (KiCad board)
At the start: 2 copper layers, 6 parts, among them P1 HEADER_8X1, P2 HEADER_8X1

Commit message: Added board edge
Other:
- board outline added: 27.9 x 25.4 mm
Changed lines of the file:
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@@
     (links 32)
     (no_connects 0)
-    (area 0 0 0 0)
+    (area 182.051 105.875445 209.109 132.884555)
     (thickness 1.6)
-    (drawings 36)
+    (drawings 40)
     (tracks 64)
     (zones 0)
@@
     )
   )
+  (gr_line (start 181.61 132.08) (end 209.55 132.08) (angle 90) (layer Edge.Cuts) (width 0.1))
+  (gr_line (start 181.61 106.68) (end 181.61 132.08) (angle 90) (layer Edge.Cuts) (width 0.1))
+  (gr_line (start 209.55 106.68) (end 181.61 106.68) (angle 90) (layer Edge.Cuts) (width 0.1))
+  (gr_line (start 209.55 132.08) (end 209.55 106.68) (angle 90) (layer Edge.Cuts) (width 0.1))
   (gr_line (start 189.23 119.38) (end 191.77 119.38) (angle 90) (layer B.SilkS) (width 0.2))
   (gr_line (start 189.23 127) (end 191.77 127) (angle 90) (layer B.SilkS) (width 0.2))
